File: pcb/GoL 1.3.brd (EAGLE design)
At the start: 71.1 x 71.1 mm, 43 parts, among them IC1 ATMEGA48-10PI

Commit message: Finished routing
Parts:
- removed C3: 0.1uF, rcl-ez:C025-025X050
- removed E, N, S, W: CONNECT4, lifeofrush:CON4-0.15
- removed ICSP: (no value), pinhead:2X03
- added SV1, SV2, SV3, SV4: (no value), con-lstb:MA04-1
- moved C1 37.8 mm to (17.8, 4.83), turned to 180 degrees
- moved C2 25.1 mm to (36.3, 26.5)
- moved PWR 6.10 mm to (17.8, 9.78)
- moved ON/OFF 0.51 mm to (18.5, 66.5)
- moved R1 0.25 mm to (8.64, 57.1), turned to 0 degrees
Connections:
- net BCAST: now also SV1.2, SV2.2, SV3.3, SV4.3; no longer E.B3, E.F3, N.B2, N.F2, S.B3, S.F3, W.B2, W.F2
- net ERX: now also SV4.2; no longer E.B2, E.F2
- net GND: now also SV1.4, SV2.4, SV3.4, SV4.4; no longer C3.2, E.B4, E.F4, ICSP.6, N.B4, N.F4, S.B4, S.F4, W.B4, W.F4
- net MISO: no longer ICSP.1
- net MOSI: no longer ICSP.4
- net NRX: now also SV2.3; no longer N.B3, N.F3
- net RESET: no longer ICSP.5
- net SCK: no longer ICSP.3
- net SRX: now also SV3.2; no longer S.B2, S.F2
- net V+: now also SV1.1, SV2.1, SV3.1, SV4.1; no longer C3.1, E.B1, E.F1, ICSP.2, N.B1, N.F1, S.B1, S.F1, W.B1, W.F1
- net WRX: now also SV1.3; no longer W.B3, W.F3
Routing:
- net GND: track 416.3 -> 0.00 mm, vias 4 -> 0
- net MOSI: track 128.8 -> 29.5 mm, vias 2 -> 0
- net BCAST: track 267.9 -> 170.4 mm, vias 7 -> 2
- net MISO: track 104.4 -> 41.0 mm
- net N$26: track 63.3 -> 115.9 mm, vias 1 -> 0
- net V+: track 307.1 -> 260.8 mm, vias 5 -> 0
- net SCK: track 56.8 -> 21.8 mm
- net N$27: track 75.8 -> 43.9 mm
- net N$28: track 20.5 -> 51.0 mm
- net RESET: track 19.0 -> 0.00 mm
- net N$20: track 57.2 -> 40.3 mm
- net N$18: track 27.7 -> 38.9 mm
- net N$33: track 42.0 -> 32.2 mm
- net WRX: track 33.8 -> 24.8 mm, vias 1 -> 0
- net N$21: track 36.3 -> 27.5 mm
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- added copper zone on layer 16, net GND
Other:
- board text added: "Game of Life"
- board text added: "THOR"
- board text removed: "3-5VDC"
- board text removed: "Game of Life v1.3"
