File: pcb/GoL 1.3.sch (EAGLE design)
At the start: 43 parts, among them IC1 ATMEGA48-10PI

Commit message: Finished routing
Parts:
- removed C3: 0.1uF, rcl-ez:C-US025-025X050
- removed E, N, S, W: CONNECT4, lifeofrush:CONNECT4
- removed ICSP: (no value), pinhead:PINHD-2X3
- added SV1, SV2, SV3, SV4: (no value), con-lstb:MA04-1
Connections:
- net BCAST: now also SV1.2, SV2.2, SV3.3, SV4.3; no longer E.B3, E.F3, N.B2, N.F2, S.B3, S.F3, W.B2, W.F2
- net ERX: now also SV4.2; no longer E.B2, E.F2
- net GND: now also SV1.4, SV2.4, SV3.4, SV4.4; no longer C3.2, E.B4, E.F4, ICSP.6, N.B4, N.F4, S.B4, S.F4, W.B4, W.F4
- net MISO: no longer ICSP.1
- net MOSI: no longer ICSP.4
- net NRX: now also SV2.3; no longer N.B3, N.F3
- net RESET: no longer ICSP.5
- net SCK: no longer ICSP.3
- net SRX: now also SV3.2; no longer S.B2, S.F2
- net V+: now also SV1.1, SV2.1, SV3.1, SV4.1; no longer C3.1, E.B1, E.F1, ICSP.2, N.B1, N.F1, S.B1, S.F1, W.B1, W.F1
- net WRX: now also SV1.3; no longer W.B3, W.F3
